Commit message: towards gemma setup

File: ur_moveit_config/srdf/ur_macro.srdf.xacro (robot description, xacro)
@@ -39,4 +39,68 @@
       <joint name="${prefix}wrist_3_joint" value="-0.11" />
     </group_state>
+    <group_state name="${prefix}calibrating_airbrush_position" group="${prefix}${name}_manipulator">
+        <joint name="${prefix}shoulder_pan_joint"    value="1.344" />
+        <joint name="${prefix}shoulder_lift_joint"   value="-0.9519" />
+        <joint name="${prefix}elbow_joint"           value="0.902" />
+        <joint name="${prefix}wrist_1_joint"         value="0.07" />
+        <joint name="${prefix}wrist_2_joint"         value="1.326" />
+        <joint name="${prefix}wrist_3_joint"         value="-3.14159" />
+    </group_state>
+    <group_state name="${prefix}calibrating_static_camera_position" group="${prefix}${name}_manipulator">
+        <joint name="${prefix}shoulder_pan_joint"    value="1.2939" />
+        <joint name="${prefix}shoulder_lift_joint"   value="-1.3631" />
+        <joint name="${prefix}elbow_joint"           value="0.9788" />
+        <joint name="${prefix}wrist_1_joint"         value="-1.5643" />
+        <joint name="${prefix}wrist_2_joint"         value="-1.5383" />
+        <joint name="${prefix}wrist_3_joint"         value="-0.2405" />
+    </group_state>
+    <group_state name="${prefix}paint_calib_position" group="${prefix}${name}_manipulator">
+        <joint name="${prefix}shoulder_pan_joint"    value="0.0174" />
+        <joint name="${prefix}shoulder_lift_joint"   value="-2.088" />
+        <joint name="${prefix}elbow_joint"           value="1.9488" />
+        <joint name="${prefix}wrist_1_joint"         value="0.1914" />
+        <joint name="${prefix}wrist_2_joint"         value="1.5834" />
+        <joint name="${prefix}wrist_3_joint"         value="-3.1146" />
+    </group_state>
+    <group_state name="${prefix}forward_scan_position" group="${prefix}${name}_manipulator">
+        <joint name="${prefix}shoulder_pan_joint"    value="1.229" />
+        <joint name="${prefix}shoulder_lift_joint"   value="-1.759" />
+        <joint name="${prefix}elbow_joint"           value="1.969" />
+        <joint name="${prefix}wrist_1_joint"         value="-0.251" />
+        <joint name="${prefix}wrist_2_joint"         value="1.253" />
+        <joint name="${prefix}wrist_3_joint"         value="-3.141" />
+    </group_state>
+    <group_state name="${prefix}left_scan_position" group="${prefix}${name}_manipulator">
+        <joint name="${prefix}shoulder_pan_joint"    value="0" />
+        <joint name="${prefix}shoulder_lift_joint"   value="0" />
+        <joint name="${prefix}elbow_joint"           value="0" />
+        <joint name="${prefix}wrist_1_joint"         value="1" />
+        <joint name="${prefix}wrist_2_joint"         value="1" />
+        <joint name="${prefix}wrist_3_joint"         value="1" />
+    </group_state>
+    <group_state name="${prefix}right_scan_position" group="${prefix}${name}_manipulator">
+        <joint name="${prefix}shoulder_pan_joint"    value="0" />
+        <joint name="${prefix}shoulder_lift_joint"   value="0" />
+        <joint name="${prefix}elbow_joint"           value="0" />
+        <joint name="${prefix}wrist_1_joint"         value="1" />
+        <joint name="${prefix}wrist_2_joint"         value="1" />
+        <joint name="${prefix}wrist_3_joint"         value="1" />
+    </group_state>
+    <group_state name="${prefix}initial_guess1" group="${prefix}${name}_manipulator">
+        <joint name="${prefix}shoulder_pan_joint"    value="1.5707" />
+        <joint name="${prefix}shoulder_lift_joint"   value="-1.5707" />
+        <joint name="${prefix}elbow_joint"           value="0" />
+        <joint name="${prefix}wrist_1_joint"         value="0" />
+        <joint name="${prefix}wrist_2_joint"         value="0" />
+        <joint name="${prefix}wrist_3_joint"         value="0" />
+    </group_state>
+     <group_state name="${prefix}initial_guess2" group="${prefix}${name}_manipulator">
+        <joint name="${prefix}shoulder_pan_joint"    value="-1.5707" />
+        <joint name="${prefix}shoulder_lift_joint"   value="-1.5707" />
+        <joint name="${prefix}elbow_joint"           value="0" />
+        <joint name="${prefix}wrist_1_joint"         value="0" />
+        <joint name="${prefix}wrist_2_joint"         value="0" />
+        <joint name="${prefix}wrist_3_joint"         value="0" />
+    </group_state>
     <!--END EFFECTOR - Purpose - Represent information about an end effector.-->
     <!--VIRTUAL JOINT - Purpose - this element defines a virtual joint between a robot link and an external frame of reference (considered fixed with respect to the robot)-->
@@ -44,4 +108,5 @@
     <disable_collisions link1="${prefix}base_link" link2="${prefix}base_link_inertia" reason="Adjacent" />
     <disable_collisions link1="${prefix}base_link_inertia" link2="${prefix}shoulder_link" reason="Adjacent" />
+    <disable_collisions link1="${prefix}base_link_inertia" link2="${prefix}table" reason="Adjacent" />
     <disable_collisions link1="${prefix}tool0" link2="${prefix}wrist_1_link" reason="Never" />
     <disable_collisions link1="${prefix}tool0" link2="${prefix}wrist_2_link" reason="Never" />
@@ -53,4 +118,5 @@
     <disable_collisions link1="${prefix}wrist_1_link" link2="${prefix}wrist_3_link" reason="Never" />
     <disable_collisions link1="${prefix}wrist_2_link" link2="${prefix}wrist_3_link" reason="Adjacent" />
+    <disable_collisions link1="${prefix}wrist_3_link" link2="${prefix}tool_temp" reason="Adjacent" />
   </xacro:macro>
 </robot>

Commit message: .

File: ur_moveit_config/srdf/ur_macro.srdf.xacro (robot description, xacro)
@@ -64,9 +64,9 @@
     </group_state>
     <group_state name="${prefix}forward_scan_position" group="${prefix}${name}_manipulator">
-        <joint name="${prefix}shoulder_pan_joint"    value="1.229" />
-        <joint name="${prefix}shoulder_lift_joint"   value="-1.759" />
-        <joint name="${prefix}elbow_joint"           value="1.969" />
-        <joint name="${prefix}wrist_1_joint"         value="-0.251" />
-        <joint name="${prefix}wrist_2_joint"         value="1.253" />
+        <joint name="${prefix}shoulder_pan_joint"    value="1.2" />
+        <joint name="${prefix}shoulder_lift_joint"   value="-1.78" />
+        <joint name="${prefix}elbow_joint"           value="2.111" />
+        <joint name="${prefix}wrist_1_joint"         value="-0.349" />
+        <joint name="${prefix}wrist_2_joint"         value="1.222" />
         <joint name="${prefix}wrist_3_joint"         value="-3.141" />
     </group_state>

Commit message: .

File: ur_moveit_config/srdf/ur_macro.srdf.xacro (robot description, xacro)
@@ -38,4 +38,12 @@
       <joint name="${prefix}wrist_2_joint" value="-1.6" />
       <joint name="${prefix}wrist_3_joint" value="-0.11" />
+    </group_state>
+    <group_state name="${prefix}eih_calib_scan_position" group="${prefix}${name}_manipulator">
+        <joint name="${prefix}shoulder_pan_joint"    value="1.2" />
+        <joint name="${prefix}shoulder_lift_joint"   value="-1.78" />
+        <joint name="${prefix}elbow_joint"           value="2.111" />
+        <joint name="${prefix}wrist_1_joint"         value="-0.349" />
+        <joint name="${prefix}wrist_2_joint"         value="1.222" />
+        <joint name="${prefix}wrist_3_joint"         value="-3.141" />
     </group_state>
     <group_state name="${prefix}calibrating_airbrush_position" group="${prefix}${name}_manipulator">

Commit message: .

File: ur_moveit_config/srdf/ur_macro.srdf.xacro (robot description, xacro)
@@ -46,4 +46,12 @@
         <joint name="${prefix}wrist_2_joint"         value="1.222" />
         <joint name="${prefix}wrist_3_joint"         value="-3.141" />
+    </group_state>
+    <group_state name="${prefix}eob_calib_scan_position" group="${prefix}${name}_manipulator">
+        <joint name="${prefix}shoulder_pan_joint"    value="-1.29" />
+        <joint name="${prefix}shoulder_lift_joint"   value="-2.356" />
+        <joint name="${prefix}elbow_joint"           value="-0.139" />
+        <joint name="${prefix}wrist_1_joint"         value="-1.884" />
+        <joint name="${prefix}wrist_2_joint"         value="1.274" />
+        <joint name="${prefix}wrist_3_joint"         value="3.089" />
     </group_state>
     <group_state name="${prefix}calibrating_airbrush_position" group="${prefix}${name}_manipulator">

Commit message: .

File: ur_moveit_config/srdf/ur_macro.srdf.xacro (robot description, xacro)
@@ -79,5 +79,29 @@
         <joint name="${prefix}wrist_3_joint"         value="-3.1146" />
     </group_state>
-    <group_state name="${prefix}forward_scan_position" group="${prefix}${name}_manipulator">
+    <group_state name="${prefix}forward_scan_position1" group="${prefix}${name}_manipulator">
+        <joint name="${prefix}shoulder_pan_joint"    value="1.2" />
+        <joint name="${prefix}shoulder_lift_joint"   value="-1.78" />
+        <joint name="${prefix}elbow_joint"           value="2.111" />
+        <joint name="${prefix}wrist_1_joint"         value="-0.349" />
+        <joint name="${prefix}wrist_2_joint"         value="1.222" />
+        <joint name="${prefix}wrist_3_joint"         value="-3.141" />
+    </group_state>
+    <group_state name="${prefix}forward_scan_position2" group="${prefix}${name}_manipulator">
+        <joint name="${prefix}shoulder_pan_joint"    value="1.2" />
+        <joint name="${prefix}shoulder_lift_joint"   value="-1.78" />
+        <joint name="${prefix}elbow_joint"           value="2.111" />
+        <joint name="${prefix}wrist_1_joint"         value="-0.349" />
+        <joint name="${prefix}wrist_2_joint"         value="1.222" />
+        <joint name="${prefix}wrist_3_joint"         value="-3.141" />
+    </group_state>
+    <group_state name="${prefix}forward_scan_position3" group="${prefix}${name}_manipulator">
+        <joint name="${prefix}shoulder_pan_joint"    value="1.2" />
+        <joint name="${prefix}shoulder_lift_joint"   value="-1.78" />
+        <joint name="${prefix}elbow_joint"           value="2.111" />
+        <joint name="${prefix}wrist_1_joint"         value="-0.349" />
+        <joint name="${prefix}wrist_2_joint"         value="1.222" />
+        <joint name="${prefix}wrist_3_joint"         value="-3.141" />
+    </group_state>
+    <group_state name="${prefix}forward_scan_position4" group="${prefix}${name}_manipulator">
         <joint name="${prefix}shoulder_pan_joint"    value="1.2" />
         <joint name="${prefix}shoulder_lift_joint"   value="-1.78" />

Commit message: .

File: ur_moveit_config/srdf/ur_macro.srdf.xacro (robot description, xacro)
@@ -78,4 +78,12 @@
         <joint name="${prefix}wrist_2_joint"         value="1.5834" />
         <joint name="${prefix}wrist_3_joint"         value="-3.1146" />
+    </group_state>
+    <group_state name="${prefix}rest_position" group="${prefix}${name}_manipulator">
+        <joint name="${prefix}shoulder_pan_joint"    value="1.2" />
+        <joint name="${prefix}shoulder_lift_joint"   value="-1.78" />
+        <joint name="${prefix}elbow_joint"           value="2.111" />
+        <joint name="${prefix}wrist_1_joint"         value="-0.349" />
+        <joint name="${prefix}wrist_2_joint"         value="1.222" />
+        <joint name="${prefix}wrist_3_joint"         value="-3.141" />
     </group_state>
     <group_state name="${prefix}forward_scan_position1" group="${prefix}${name}_manipulator">

Commit message: .

File: ur_moveit_config/srdf/ur_macro.srdf.xacro (robot description, xacro)
@@ -87,29 +87,5 @@
         <joint name="${prefix}wrist_3_joint"         value="-3.141" />
     </group_state>
-    <group_state name="${prefix}forward_scan_position1" group="${prefix}${name}_manipulator">
-        <joint name="${prefix}shoulder_pan_joint"    value="1.2" />
-        <joint name="${prefix}shoulder_lift_joint"   value="-1.78" />
-        <joint name="${prefix}elbow_joint"           value="2.111" />
-        <joint name="${prefix}wrist_1_joint"         value="-0.349" />
-        <joint name="${prefix}wrist_2_joint"         value="1.222" />
-        <joint name="${prefix}wrist_3_joint"         value="-3.141" />
-    </group_state>
-    <group_state name="${prefix}forward_scan_position2" group="${prefix}${name}_manipulator">
-        <joint name="${prefix}shoulder_pan_joint"    value="1.2" />
-        <joint name="${prefix}shoulder_lift_joint"   value="-1.78" />
-        <joint name="${prefix}elbow_joint"           value="2.111" />
-        <joint name="${prefix}wrist_1_joint"         value="-0.349" />
-        <joint name="${prefix}wrist_2_joint"         value="1.222" />
-        <joint name="${prefix}wrist_3_joint"         value="-3.141" />
-    </group_state>
-    <group_state name="${prefix}forward_scan_position3" group="${prefix}${name}_manipulator">
-        <joint name="${prefix}shoulder_pan_joint"    value="1.2" />
-        <joint name="${prefix}shoulder_lift_joint"   value="-1.78" />
-        <joint name="${prefix}elbow_joint"           value="2.111" />
-        <joint name="${prefix}wrist_1_joint"         value="-0.349" />
-        <joint name="${prefix}wrist_2_joint"         value="1.222" />
-        <joint name="${prefix}wrist_3_joint"         value="-3.141" />
-    </group_state>
-    <group_state name="${prefix}forward_scan_position4" group="${prefix}${name}_manipulator">
+    <group_state name="${prefix}forward_scan_position" group="${prefix}${name}_manipulator">
         <joint name="${prefix}shoulder_pan_joint"    value="1.2" />
         <joint name="${prefix}shoulder_lift_joint"   value="-1.78" />

Commit message: .

File: ur_moveit_config/srdf/ur_macro.srdf.xacro (robot description, xacro)
@@ -47,5 +47,37 @@
         <joint name="${prefix}wrist_3_joint"         value="-3.141" />
     </group_state>
-    <group_state name="${prefix}eob_calib_scan_position" group="${prefix}${name}_manipulator">
+    <group_state name="${prefix}eob_calib_scan_position1" group="${prefix}${name}_manipulator">
+        <joint name="${prefix}shoulder_pan_joint"    value="-1.29" />
+        <joint name="${prefix}shoulder_lift_joint"   value="-2.356" />
+        <joint name="${prefix}elbow_joint"           value="-0.139" />
+        <joint name="${prefix}wrist_1_joint"         value="-1.884" />
+        <joint name="${prefix}wrist_2_joint"         value="1.274" />
+        <joint name="${prefix}wrist_3_joint"         value="3.089" />
+    </group_state>
+    <group_state name="${prefix}eob_calib_scan_position2" group="${prefix}${name}_manipulator">
+        <joint name="${prefix}shoulder_pan_joint"    value="-1.29" />
+        <joint name="${prefix}shoulder_lift_joint"   value="-2.356" />
+        <joint name="${prefix}elbow_joint"           value="-0.139" />
+        <joint name="${prefix}wrist_1_joint"         value="-1.884" />
+        <joint name="${prefix}wrist_2_joint"         value="1.274" />
+        <joint name="${prefix}wrist_3_joint"         value="3.089" />
+    </group_state>
+    <group_state name="${prefix}eob_calib_scan_position3" group="${prefix}${name}_manipulator">
+        <joint name="${prefix}shoulder_pan_joint"    value="-1.29" />
+        <joint name="${prefix}shoulder_lift_joint"   value="-2.356" />
+        <joint name="${prefix}elbow_joint"           value="-0.139" />
+        <joint name="${prefix}wrist_1_joint"         value="-1.884" />
+        <joint name="${prefix}wrist_2_joint"         value="1.274" />
+        <joint name="${prefix}wrist_3_joint"         value="3.089" />
+    </group_state>
+    <group_state name="${prefix}eob_calib_scan_position4" group="${prefix}${name}_manipulator">
+        <joint name="${prefix}shoulder_pan_joint"    value="-1.29" />
+        <joint name="${prefix}shoulder_lift_joint"   value="-2.356" />
+        <joint name="${prefix}elbow_joint"           value="-0.139" />
+        <joint name="${prefix}wrist_1_joint"         value="-1.884" />
+        <joint name="${prefix}wrist_2_joint"         value="1.274" />
+        <joint name="${prefix}wrist_3_joint"         value="3.089" />
+    </group_state>
+    <group_state name="${prefix}eob_calib_scan_position5" group="${prefix}${name}_manipulator">
         <joint name="${prefix}shoulder_pan_joint"    value="-1.29" />
         <joint name="${prefix}shoulder_lift_joint"   value="-2.356" />

Commit message: .

File: ur_moveit_config/srdf/ur_macro.srdf.xacro (robot description, xacro)
@@ -119,5 +119,13 @@
         <joint name="${prefix}wrist_3_joint"         value="-3.141" />
     </group_state>
-    <group_state name="${prefix}forward_scan_position" group="${prefix}${name}_manipulator">
+    <group_state name="${prefix}forward_scan_position_close" group="${prefix}${name}_manipulator">
+        <joint name="${prefix}shoulder_pan_joint"    value="1.2" />
+        <joint name="${prefix}shoulder_lift_joint"   value="-1.78" />
+        <joint name="${prefix}elbow_joint"           value="2.111" />
+        <joint name="${prefix}wrist_1_joint"         value="-0.349" />
+        <joint name="${prefix}wrist_2_joint"         value="1.222" />
+        <joint name="${prefix}wrist_3_joint"         value="-3.141" />
+    </group_state>
+    <group_state name="${prefix}forward_scan_position_far" group="${prefix}${name}_manipulator">
         <joint name="${prefix}shoulder_pan_joint"    value="1.2" />
         <joint name="${prefix}shoulder_lift_joint"   value="-1.78" />

Commit message: .

File: ur_moveit_config/srdf/ur_macro.srdf.xacro (robot description, xacro)
@@ -87,4 +87,44 @@
         <joint name="${prefix}wrist_3_joint"         value="3.089" />
     </group_state>
+    <group_state name="${prefix}eob_calib_scan_position6" group="${prefix}${name}_manipulator">
+        <joint name="${prefix}shoulder_pan_joint"    value="-1.29" />
+        <joint name="${prefix}shoulder_lift_joint"   value="-2.356" />
+        <joint name="${prefix}elbow_joint"           value="-0.139" />
+        <joint name="${prefix}wrist_1_joint"         value="-1.884" />
+        <joint name="${prefix}wrist_2_joint"         value="1.274" />
+        <joint name="${prefix}wrist_3_joint"         value="3.089" />
+    </group_state>
+    <group_state name="${prefix}eob_calib_scan_position7" group="${prefix}${name}_manipulator">
+        <joint name="${prefix}shoulder_pan_joint"    value="-1.29" />
+        <joint name="${prefix}shoulder_lift_joint"   value="-2.356" />
+        <joint name="${prefix}elbow_joint"           value="-0.139" />
+        <joint name="${prefix}wrist_1_joint"         value="-1.884" />
+        <joint name="${prefix}wrist_2_joint"         value="1.274" />
+        <joint name="${prefix}wrist_3_joint"         value="3.089" />
+    </group_state>
+    <group_state name="${prefix}eob_calib_scan_position8" group="${prefix}${name}_manipulator">
+        <joint name="${prefix}shoulder_pan_joint"    value="-1.29" />
+        <joint name="${prefix}shoulder_lift_joint"   value="-2.356" />
+        <joint name="${prefix}elbow_joint"           value="-0.139" />
+        <joint name="${prefix}wrist_1_joint"         value="-1.884" />
+        <joint name="${prefix}wrist_2_joint"         value="1.274" />
+        <joint name="${prefix}wrist_3_joint"         value="3.089" />
+    </group_state>
+    <group_state name="${prefix}eob_calib_scan_position9" group="${prefix}${name}_manipulator">
+        <joint name="${prefix}shoulder_pan_joint"    value="-1.29" />
+        <joint name="${prefix}shoulder_lift_joint"   value="-2.356" />
+        <joint name="${prefix}elbow_joint"           value="-0.139" />
+        <joint name="${prefix}wrist_1_joint"         value="-1.884" />
+        <joint name="${prefix}wrist_2_joint"         value="1.274" />
+        <joint name="${prefix}wrist_3_joint"         value="3.089" />
+    </group_state>
+    <group_state name="${prefix}eob_calib_scan_position10" group="${prefix}${name}_manipulator">
+        <joint name="${prefix}shoulder_pan_joint"    value="-1.29" />
+        <joint name="${prefix}shoulder_lift_joint"   value="-2.356" />
+        <joint name="${prefix}elbow_joint"           value="-0.139" />
+        <joint name="${prefix}wrist_1_joint"         value="-1.884" />
+        <joint name="${prefix}wrist_2_joint"         value="1.274" />
+        <joint name="${prefix}wrist_3_joint"         value="3.089" />
+    </group_state>
     <group_state name="${prefix}calibrating_airbrush_position" group="${prefix}${name}_manipulator">
         <joint name="${prefix}shoulder_pan_joint"    value="1.344" />
